File: FOC_V1_PCB/power_mosfet.kicad_sch (KiCad schematic)
At the start: 8 parts, among them U3 IRFS7530TRL7PP, U4 IRFS7530TRL7PP, U5 IRFS7530TRL7PP, U6 IRFS7530TRL7PP, U7 IRFS7530TRL7PP, U8 IRFS7530TRL7PP

Commit message: new V1.2 PCB and tweaked mechanical rig
Connections:
- net DRV_SH_A: now also U3.7 (S); no longer U6.7 (D)
- net DRV_SH_B: now also U4.7 (S); no longer U7.7 (D)
- net DRV_SH_C: now also U5.7 (S); no longer U8.7 (D)
- net DRV_SL_A: now also U6.7 (S)
- net DRV_SL_C: now also U8.7 (S)
- net GND: now also U7.7 (S)
- net V_Supply_+42V: no longer U3.7 (D), U4.7 (D), U5.7 (D)
Other:
- note added: "Must route it using a Kelvin Connection: Dedicated Traces: Draw a thin, dedicated trace directly from the SP1 pin to the physical copper pad on the inside edge of the upper side of the shunt resistor. Do the same for Ground: Draw another thin, dedicated trace directly from the SN1 pin to the physical copper pad on the inside edge of the bottom side of the shunt resistor. Do NOT connect SN1 to you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"
- note removed: "You must route it using a Kelvin Connection: Dedicated Traces: Draw a thin, dedicated trace directly from the SP1 pin to the physical copper pad on the inside edge of the upper side of the shunt resistor. Do the same for Ground: Draw another thin, dedicated trace directly from the SN1 pin to the physical copper pad on the inside edge of the bottom side of the shunt resistor. Do NOT connect SN1 to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"
Changed lines of the file:
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@@
 	(generator_version "10.0")
 	(paper "A4")
-	(text "You must route it using a Kelvin Connection:\n\nDedicated Traces: Draw a thin, dedicated trace directly \nfrom the SP1 pin to the physical copper pad on the \ninside edge of the upper side of the shunt resistor.\n\nDo the same for Ground: Draw another thin, dedicated trace \ndirectly from the SN1 pin to the physical copper pad on the \ninside edge of the bottom side of the shunt resistor. \nDo NOT connect SN1 to your main ground plane anywhere else \nit must only touch ground right at the resistor pad.\n\nRoute them together: \nRoute the SP1 and SN1 traces right next to each other, parallel, \nall the way from the DRV8301 to the resistor. \nThis is called a Differential Pair. \nBecause they are right next to each other, \nany magnetic noise from the motor will hit both wires equally, \nand the DRV8301's amplifier will magically cancel the noise out!"
+	(text "Must route it using a Kelvin Connection:\n\nDedicated Traces: Draw a thin, dedicated trace directly \nfrom the SP1 pin to the physical copper pad on the \ninside edge of the upper side of the shunt resistor.\n\nDo the same for Ground: Draw another thin, dedicated trace \ndirectly from the SN1 pin to the physical copper pad on the \ninside edge of the bottom side of the shunt resistor. \nDo NOT connect SN1 to your main ground plane anywhere else \nit must only touch ground right at the resistor pad.\n\nRoute them together: \nRoute the SP1 and SN1 traces right next to each other, parallel, \nall the way from the DRV8301 to the resistor. \nThis is called a Differential Pair. \nBecause they are right next to each other, \nany magnetic noise from the motor will hit both wires equally, \nand the DRV8301's amplifier will magically cancel the noise out!"
 		(exclude_from_sim no)
 		(at 135.636 147.32 0)
@@
 	)
 	(junction
-		(at 157.48 67.31)
-		(diameter 0)
-		(color 0 0 0 0)
-	)
-	(junction
-		(at 83.82 101.6)
-		(diameter 0)
-		(color 0 0 0 0)
-	)
-	(junction
 		(at 229.87 115.57)
 		(diameter 0)
@@
 	)
 	(junction
+		(at 83.82 72.39)
+		(diameter 0)
+		(color 0 0 0 0)
+	)
+	(junction
 		(at 157.48 109.22)
 		(diameter 0)
@@
 	)
 	(junction
-		(at 157.48 101.6)
-		(diameter 0)
-		(color 0 0 0 0)
-	)
-	(junction
 		(at 83.82 81.28)
 		(diameter 0)
@@
 	)
 	(junction
-		(at 83.82 67.31)
+		(at 229.87 106.68)
 		(diameter 0)
 		(color 0 0 0 0)
@@
 	)
 	(junction
+		(at 157.48 72.39)
+		(diameter 0)
+		(color 0 0 0 0)
+	)
+	(junction
 		(at 40.64 106.68)
 		(diameter 0)
@@
 	)
 	(junction
+		(at 229.87 73.66)
+		(diameter 0)
+		(color 0 0 0 0)
+	)
+	(junction
 		(at 114.3 74.93)
 		(diameter 0)
@@
 	)
 	(junction
-		(at 229.87 68.58)
-		(diameter 0)
-		(color 0 0 0 0)
-	)
-	(junction
 		(at 186.69 106.68)
 		(diameter 0)
@@
 	)
 	(junction
-		(at 229.87 101.6)
+		(at 83.82 106.68)
 		(diameter 0)
 		(color 0 0 0 0)
@@
 	)
 	(junction
+		(at 157.48 106.68)
+		(diameter 0)
+		(color 0 0 0 0)
+	)
+	(junction
 		(at 186.69 76.2)
 		(diameter 0)
@@
 	(wire
 		(pts
-			(xy 83.82 67.31) (xy 83.82 69.85)
+			(xy 157.48 69.85) (xy 157.48 72.39)
 		)
 		(stroke
@@
 	(wire
 		(pts
+			(xy 83.82 104.14) (xy 83.82 106.68)
+		)
+		(stroke
+			(width 0)
+			(type default)
+		)
+	)
+	(wire
+		(pts
 			(xy 157.48 115.57) (xy 157.48 109.22)
 		)
@@
 	(wire
 		(pts
-			(xy 157.48 67.31) (xy 157.48 69.85)
-		)
-		(stroke
-			(width 0)
-			(type default)
-		)
-	)
-	(wire
-		(pts
 			(xy 157.48 109.22) (xy 157.48 106.68)
 		)
@@
 	(wire
 		(pts
+			(xy 229.87 71.12) (xy 229.87 73.66)
+		)
+		(stroke
+			(width 0)
+			(type default)
+		)
+	)
+	(wire
+		(pts
+			(xy 83.82 69.85) (xy 83.82 72.39)
+		)
+		(stroke
+			(width 0)
+			(type default)
+		)
+	)
+	(wire
+		(pts
 			(xy 40.64 69.85) (xy 40.64 72.39)
 		)
@@
 	(wire
 		(pts
-			(xy 83.82 101.6) (xy 83.82 104.14)
-		)
-		(stroke
-			(width 0)
-			(type default)
-		)
-	)
-	(wire
-		(pts
 			(xy 83.82 74.93) (xy 83.82 72.39)
 		)
@@
 	(wire
 		(pts
+			(xy 229.87 104.14) (xy 229.87 106.68)
+		)
+		(stroke
+			(width 0)
+			(type default)
+		)
+	)
+	(wire
+		(pts
 			(xy 157.48 81.28) (xy 157.48 88.9)
 		)
@@
 	(wire
 		(pts
-			(xy 229.87 101.6) (xy 229.87 104.14)
-		)
-		(stroke
-			(width 0)
-			(type default)
-		)
-	)
-	(wire
-		(pts
 			(xy 229.87 73.66) (xy 228.6 73.66)
 		)
@@
 	(wire
 		(pts
+			(xy 157.48 104.14) (xy 157.48 106.68)
+		)
+		(stroke
+			(width 0)
+			(type default)
+		)
+	)
+	(wire
+		(pts
 			(xy 187.96 104.14) (xy 186.69 104.14)
 		)
@@
 	(wire
 		(pts
-			(xy 229.87 68.58) (xy 229.87 71.12)
-		)
-		(stroke
-			(width 0)
-			(type default)
-		)
-	)
-	(wire
-		(pts
 			(xy 114.3 74.93) (xy 114.3 81.28)
 		)
@@
 		(pts
 			(xy 82.55 109.22) (xy 83.82 109.22)
-		)
-		(stroke
-			(width 0)
-			(type default)
-		)
-	)
-	(wire
-		(pts
-			(xy 157.48 101.6) (xy 157.48 104.14)
 		)
 		(stroke
@@
 	)
 	(symbol
+		(lib_name "IRFS7530TRL7PP_4")
 		(lib_id "FOC_sym_lib:IRFS7530TRL7PP")
 		(at 41.91 101.6 0)
@@
 	)
 	(symbol
+		(lib_name "IRFS7530TRL7PP_2")
 		(lib_id "FOC_sym_lib:IRFS7530TRL7PP")
 		(at 115.57 67.31 0)
@@
 	)
 	(symbol
+		(lib_name "IRFS7530TRL7PP_5")
 		(lib_id "FOC_sym_lib:IRFS7530TRL7PP")
 		(at 115.57 101.6 0)
@@
 	)
 	(symbol
+		(lib_name "IRFS7530TRL7PP_3")
 		(lib_id "FOC_sym_lib:IRFS7530TRL7PP")
 		(at 187.96 68.58 0)
@@
 	)
 	(symbol
+		(lib_name "IRFS7530TRL7PP_1")
 		(lib_id "FOC_sym_lib:IRFS7530TRL7PP")
 		(at 41.91 67.31 0)
