File: FOC_V1_PCB/FOC_V1_PCB.kicad_pcb (KiCad board)
At the start: 4 copper layers, 112.9 x 72.6 mm, 105 parts, among them J1 ST-Link_01x05, J10 C, J2 Enc_MCU_01x06, J3 Enc_Enc_01x06, J4 CAN_01x04, J6 +V, J7 GND, J8 A, J9 B, SW1 TS-1002S-05026C, U1 STM32F405RGT6, U10 TJA1051T/3/1J, U11 ME6211, U2 DRV8301DCAR, U3 IRFS7530TRL7PP, U4 IRFS7530TRL7PP, U5 IRFS7530TRL7PP, U6 IRFS7530TRL7PP, U7 IRFS7530TRL7PP, U8 IRFS7530TRL7PP, U9 AS5048A-HTSP, Y1 Crystal_GND24

Commit message: V1.1: improved clearances, connectors, and seperated FOC board with encoder board
Parts:
- removed C34: 100nF, Capacitor_SMD:C_0603_1608Metric_Pad1.08x0.95mm_HandSolder
- removed J3: Enc_Enc_01x06, Connector_PinHeader_2.00mm:PinHeader_1x06_P2.00mm_Horizontal
- removed R27: 10kΩ, Resistor_SMD:R_0603_1608Metric_Pad0.98x0.95mm_HandSolder
- removed REF**1, REF**2, REF**3, REF**4: MountingHole_3.2mm_M3_Pad, MountingHole:MountingHole_3.2mm_M3_Pad
- removed U9: AS5048A-HTSP, FOC_foot_lib:AS5048A_TSSOP14_AMS
- removed mouse-bite-2mm-slot (x2): VAL**, Mouse_Bites:mouse-bite-2mm-slot
- J2: footprint Connector_PinHeader_2.00mm:PinHeader_1x06_P2.00mm_Horizontal -> FOC_foot_lib:JST-GH_6pin_CONN_SM06B-GHS-TB_JST; moved to B.Cu
- J4: footprint Connector_PinHeader_2.00mm:PinHeader_1x04_P2.00mm_Horizontal -> FOC_foot_lib:JST-GH_4pin_CONN_SM04B-GHS-TB_JST
- moved J2 8.30 mm to (140.2, 109.4), turned to 90 degrees
- moved J4 5.58 mm to (165.4, 117.4), turned to 0 degrees
Connections:
- USB1 pad 2: GND -> (no net)
- USB1 pad 3: GND -> (no net)
- USB1 pad 4: GND -> (no net)
Routing:
- net ENC_+3.3V: track 23.2 -> 0.00 mm, vias 1 -> 0
- net SDI_ENC: track 15.2 -> 0.00 mm
- net SDO_ENC: track 14.8 -> 0.00 mm
- net SCLK_ENC: track 14.3 -> 0.00 mm
- net BUCK_+5V: track 94.4 -> 105.5 mm
- net SCS_ENC: track 10.6 -> 0.00 mm, vias 1 -> 0
- net GND_ENC: track 4.97 -> 0.00 mm, vias 13 -> 0
- net LDO_+3.3V: track 156.0 -> 160.3 mm, vias 4 -> 5
- net CAN_H: track 4.50 -> 7.92 mm
- net CAN_L: track 4.57 -> 7.59 mm, vias 0 -> 2
- net ENC_SPI_SDI: track 19.5 -> 22.4 mm, vias 1 -> 2
- net ENC_SPI_SDO: track 20.6 -> 23.0 mm, vias 1 -> 2
- net ENC_SPI_SCLK: track 21.3 -> 23.5 mm, vias 1 -> 2
- net ENC_SPI_SCS: track 29.8 -> 28.6 mm, vias 1 -> 2
- net GND: vias 103 -> 100
- removed copper zone on B.Cu, net GND_ENC
- removed copper zone on F.Cu, net GND_ENC
Other:
- board size 112.9 x 72.6 mm -> 72.6 x 72.6 mm

Commit message: new V1.2 PCB and tweaked mechanical rig
Connections:
- U3 pad 7: V_Supply_+42V -> DRV_SH_A
- U4 pad 7: V_Supply_+42V -> DRV_SH_B
- U5 pad 7: V_Supply_+42V -> DRV_SH_C
- U6 pad 7: DRV_SH_A -> DRV_SL_A
- U7 pad 7: DRV_SH_B -> GND
- U8 pad 7: DRV_SH_C -> DRV_SL_C
Routing:
- net DRV_SH_B: track 28.9 -> 40.8 mm
- net DRV_SH_C: track 50.1 -> 58.8 mm
- net DRV_GH_C: track 70.3 -> 76.5 mm
- net DRV_SH_A: track 31.6 -> 35.3 mm
- net GND: track 45.9 -> 47.0 mm

Commit message: new V1.3 design (fixed USB-C)
Connections:
- R24 pad 1: Net-(USB1-DN1) -> Net-(USB1-DP1)
- R25 pad 1: Net-(USB1-DN2) -> Net-(USB1-DN1)
- USB1 pad A6: Net-(USB1-DN1) -> Net-(USB1-DP1)
- USB1 pad B6: Net-(USB1-DN2) -> Net-(USB1-DP1)
- USB1 pad B7: Net-(USB1-DN2) -> Net-(USB1-DN1)
Routing:
- net Net-(USB1-DN2): track 5.72 -> 0.00 mm
- net Net-(USB1-DP1): track 0.00 -> 4.77 mm
- net Net-(USB1-DN1): track 2.63 -> 4.24 mm
