File: FOC_V1_PCB/FOC_V1_PCB.kicad_sch (KiCad schematic)
At the start: 34 parts, among them J1 ST-Link_01x05, J10 C, J2 Enc_MCU_01x06, J3 Enc_Enc_01x06, J4 CAN_01x04, J6 +V, J7 GND, J8 A, J9 B, U10 TJA1051T/3/1J, U11 ME6211, U9 AS5048A-HTSP

Commit message: V1.1: improved clearances, connectors, and seperated FOC board with encoder board
Parts:
- removed C34: 100nF, Capacitor_SMD:C_0603_1608Metric_Pad1.08x0.95mm_HandSolder, symbol Device:C
- removed J3: Enc_Enc_01x06, Connector_PinHeader_2.00mm:PinHeader_1x06_P2.00mm_Horizontal, symbol Connector_Generic:Conn_01x06
- removed R27: 10kΩ, Resistor_SMD:R_0603_1608Metric_Pad0.98x0.95mm_HandSolder, symbol Device:R
- removed U9: AS5048A-HTSP, FOC_foot_lib:AS5048A_TSSOP14_AMS, symbol FOC_sym_lib:AS5048A-HTSP
- J2: footprint Connector_PinHeader_2.00mm:PinHeader_1x06_P2.00mm_Horizontal -> FOC_foot_lib:JST-GH_6pin_CONN_SM06B-GHS-TB_JST
- J4: footprint Connector_PinHeader_2.00mm:PinHeader_1x04_P2.00mm_Horizontal -> FOC_foot_lib:JST-GH_4pin_CONN_SM04B-GHS-TB_JST
Connections:
- no-connect marks 10 -> 4
Other:
- note added: "JST-GH Type"
- note removed: "JST-PH Type"
- moved on the sheet: J2

Commit message: new V1.3 design (fixed USB-C)
Connections:
- net at R25.1, USB1.B7 (DN2): now also USB1.A7 (DN1); no longer USB1.B6 (DP2)
- net at R24.1, USB1.A6 (DP1): now also USB1.B6 (DP2); no longer USB1.A7 (DN1)
Changed lines of the file:
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@@
+	)
+	(junction
+		(at 209.55 46.99)
+		(diameter 0)
+		(color 0 0 0 0)
+	)
+	(junction
+		(at 30.48 138.43)
+		(diameter 0)
+		(color 0 0 0 0)
 	)
 	(junction
@@
 	)
 	(junction
-		(at 209.55 46.99)
-		(diameter 0)
-		(color 0 0 0 0)
-	)
-	(junction
-		(at 30.48 138.43)
-		(diameter 0)
-		(color 0 0 0 0)
-	)
-	(junction
 		(at 25.4 33.02)
 		(diameter 0)
@@
 	(wire
 		(pts
+			(xy 69.85 77.47) (xy 71.12 77.47)
+		)
+		(stroke
+			(width 0)
+			(type default)
+		)
+	)
+	(wire
+		(pts
 			(xy 30.48 138.43) (xy 53.34 138.43)
 		)
@@
 	(wire
 		(pts
+			(xy 73.66 80.01) (xy 73.66 96.52)
+		)
+		(stroke
+			(width 0)
+			(type default)
+		)
+	)
+	(wire
+		(pts
 			(xy 109.22 132.08) (xy 115.57 132.08)
 		)
@@
 	(wire
 		(pts
+			(xy 43.18 93.98) (xy 43.18 80.01)
+		)
+		(stroke
+			(width 0)
+			(type default)
+		)
+	)
+	(wire
+		(pts
 			(xy 63.5 40.64) (xy 63.5 44.45)
 		)
@@
 	(wire
 		(pts
-			(xy 43.18 80.01) (xy 43.18 93.98)
-		)
-		(stroke
-			(width 0)
-			(type default)
-		)
-	)
-	(wire
-		(pts
 			(xy 45.72 96.52) (xy 66.04 96.52)
 		)
@@
 	(wire
 		(pts
+			(xy 43.18 80.01) (xy 46.99 80.01)
+		)
+		(stroke
+			(width 0)
+			(type default)
+		)
+	)
+	(wire
+		(pts
 			(xy 171.45 151.13) (xy 171.45 149.86)
 		)
@@
 	(wire
 		(pts
+			(xy 71.12 93.98) (xy 71.12 77.47)
+		)
+		(stroke
+			(width 0)
+			(type default)
+		)
+	)
+	(wire
+		(pts
 			(xy 68.58 161.29) (xy 68.58 162.56)
 		)
@@
 	(wire
 		(pts
+			(xy 45.72 77.47) (xy 45.72 96.52)
+		)
+		(stroke
+			(width 0)
+			(type default)
+		)
+	)
+	(wire
+		(pts
 			(xy 20.32 35.56) (xy 34.29 35.56)
 		)
@@
 	(wire
 		(pts
-			(xy 69.85 80.01) (xy 71.12 80.01)
-		)
-		(stroke
-			(width 0)
-			(type default)
-		)
-	)
-	(wire
-		(pts
 			(xy 68.58 167.64) (xy 69.85 167.64)
 		)
@@
 	(wire
 		(pts
-			(xy 73.66 96.52) (xy 73.66 77.47)
-		)
-		(stroke
-			(width 0)
-			(type default)
-		)
-	)
-	(wire
-		(pts
 			(xy 58.42 85.09) (xy 58.42 86.36)
 		)
@@
 	(wire
 		(pts
-			(xy 71.12 80.01) (xy 71.12 93.98)
-		)
-		(stroke
-			(width 0)
-			(type default)
-		)
-	)
-	(wire
-		(pts
 			(xy 78.74 33.02) (xy 77.47 33.02)
 		)
@@
 	(wire
 		(pts
+			(xy 46.99 77.47) (xy 45.72 77.47)
+		)
+		(stroke
+			(width 0)
+			(type default)
+		)
+	)
+	(wire
+		(pts
 			(xy 43.18 106.68) (xy 43.18 105.41)
 		)
@@
 	(wire
 		(pts
-			(xy 46.99 77.47) (xy 45.72 77.47)
-		)
-		(stroke
-			(width 0)
-			(type default)
-		)
-	)
-	(wire
-		(pts
 			(xy 68.58 162.56) (xy 69.85 162.56)
 		)
@@
 	(wire
 		(pts
+			(xy 69.85 80.01) (xy 73.66 80.01)
+		)
+		(stroke
+			(width 0)
+			(type default)
+		)
+	)
+	(wire
+		(pts
 			(xy 71.12 93.98) (xy 43.18 93.98)
 		)
@@
 	(wire
 		(pts
-			(xy 73.66 77.47) (xy 69.85 77.47)
-		)
-		(stroke
-			(width 0)
-			(type default)
-		)
-	)
-	(wire
-		(pts
 			(xy 106.68 142.24) (xy 109.22 142.24)
 		)
@@
 	(wire
 		(pts
-			(xy 43.18 80.01) (xy 46.99 80.01)
-		)
-		(stroke
-			(width 0)
-			(type default)
-		)
-	)
-	(wire
-		(pts
 			(xy 213.36 114.3) (xy 213.36 115.57)
 		)
@@
 		)
 		(stroke
-			(width 0)
-			(type default)
-		)
-	)
-	(wire
-		(pts
-			(xy 45.72 77.47) (xy 45.72 96.52)
-		)
-		(stroke
